Commit message: Made three-link, two-joint robot

File: body.urdf (robot description, URDF)
Before this commit: robot robot, 1 links, 0 joints
Links:
- removed link Box
- added link BackLeg, mass 1; collision box size=1 1 1; visual box size=1 1 1
- added link FrontLeg, mass 1; collision box size=1 1 1; visual box size=1 1 1
- added link Torso, mass 1; collision box size=1 1 1; visual box size=1 1 1
Joints:
- added joint Torso_BackLeg: type revolute, parent Torso, child BackLeg, origin xyz=2 0 1 rpy=0 0 0, axis 0 1 0, limit lower=-3.14159 upper=3.14159 effort=0.0 velocity=0.0
- added joint Torso_FrontLeg: type revolute, parent Torso, child FrontLeg, origin xyz=1 0 1 rpy=0 0 0, axis 0 1 0, limit lower=-3.14159 upper=3.14159 effort=0.0 velocity=0.0

Commit message: front and back legs

File: body.urdf (robot description, URDF)
Before this commit: robot robot, 3 links, 2 joints
Links:
- link BackLeg: geometry collision box size=0.2 1 0.2; visual box size=0.2 1 0.2
- link FrontLeg: geometry collision box size=0.2 1 0.2; visual box size=0.2 1 0.2
Joints:
- joint Torso_BackLeg: origin xyz=2 0 1 rpy=0 0 0 -> xyz=0 -0.5 1 rpy=0 0 0
- joint Torso_FrontLeg: origin xyz=1 0 1 rpy=0 0 0 -> xyz=0 0.5 1 rpy=0 0 0

Commit message: left and right legs done

File: body.urdf (robot description, URDF)
Before this commit: robot robot, 3 links, 2 joints
Links:
- added link LeftLeg, mass 1; collision box size=1 0.2 0.2; visual box size=1 0.2 0.2
- added link RightLeg, mass 1; collision box size=1 0.2 0.2; visual box size=1 0.2 0.2
Joints:
- added joint Torso_LeftLeg: type revolute, parent Torso, child LeftLeg, origin xyz=-0.5 0 1 rpy=0 0 0, axis 0 1 0, limit lower=-3.14159 upper=3.14159 effort=0.0 velocity=0.0
- added joint Torso_RightLeg: type revolute, parent Torso, child RightLeg, origin xyz=0.5 0 1 rpy=0 0 0, axis 0 1 0, limit lower=-3.14159 upper=3.14159 effort=0.0 velocity=0.0
- joint Torso_BackLeg: axis 0 1 0 -> 1 0 0
- joint Torso_FrontLeg: axis 0 1 0 -> 1 0 0

Commit message: lower legs done

File: body.urdf (robot description, URDF)
Before this commit: robot robot, 5 links, 4 joints
Links:
- added link LowerBackLeg, mass 1; collision box size=0.2 1 0.2; visual box size=0.2 1 0.2
- added link LowerFrontLeg, mass 1; collision box size=0.2 1 0.2; visual box size=0.2 1 0.2
- added link LowerLeftLeg, mass 1; collision box size=1 0.2 0.2; visual box size=1 0.2 0.2
- added link LowerRightLeg, mass 1; collision box size=1 0.2 0.2; visual box size=1 0.2 0.2
Joints:
- added joint BackLeg_LowerBackLeg: type revolute, parent BackLeg, child LowerBackLeg, origin xyz=0 -1 0 rpy=0 0 0, axis 1 0 0, limit lower=-3.14159 upper=3.14159 effort=0.0 velocity=0.0
- added joint FrontLeg_LowerFrontLeg: type revolute, parent FrontLeg, child LowerFrontLeg, origin xyz=0 1 0 rpy=0 0 0, axis 1 0 0, limit lower=-3.14159 upper=3.14159 effort=0.0 velocity=0.0
- added joint LeftLeg_LowerLeftLeg: type revolute, parent LeftLeg, child LowerLeftLeg, origin xyz=-1 0 0 rpy=0 0 0, axis 0 1 0, limit lower=-3.14159 upper=3.14159 effort=0.0 velocity=0.0
- added joint RightLeg_LowerRightLeg: type revolute, parent RightLeg, child LowerRightLeg, origin xyz=1 0 0 rpy=0 0 0, axis 0 1 0, limit lower=-3.14159 upper=3.14159 effort=0.0 velocity=0.0

Commit message: legs fixed

File: body.urdf (robot description, URDF)
Before this commit: robot robot, 9 links, 8 joints
Links:
- link LowerBackLeg: geometry collision box size=0.2 0.2 1; visual box size=0.2 0.2 1
- link LowerFrontLeg: geometry collision box size=0.2 0.2 1; visual box size=0.2 0.2 1
- link LowerLeftLeg: geometry collision box size=0.2 0.2 1; visual box size=0.2 0.2 1
- link LowerRightLeg: geometry collision box size=0.2 0.2 1; visual box size=0.2 0.2 1

Commit message: changed fitness to z position, two legs now

File: body.urdf (robot description, URDF)
Before this commit: robot robot, 9 links, 8 joints
Links:
- removed link LeftLeg
- removed link LowerLeftLeg
- removed link LowerRightLeg
- removed link RightLeg
Joints:
- removed joint LeftLeg_LowerLeftLeg
- removed joint RightLeg_LowerRightLeg
- removed joint Torso_LeftLeg
- removed joint Torso_RightLeg

Commit message: random jump, 2 legs

File: body.urdf (robot description, URDF)
Before this commit: robot robot, 5 links, 4 joints
Links:
- removed link BackLeg
- removed link FrontLeg
- removed link LowerBackLeg
- removed link LowerFrontLeg
- added link B1, mass 1; collision box size=0.2 1 0.2; visual box size=0.2 1 0.2
- added link F1, mass 1; collision box size=0.2 1 0.2; visual box size=0.2 1 0.2
- added link LB1, mass 1; collision box size=0.2 0.2 1; visual box size=0.2 0.2 1
- added link LF1, mass 1; collision box size=0.2 0.2 1; visual box size=0.2 0.2 1
Joints:
- removed joint BackLeg_LowerBackLeg
- removed joint FrontLeg_LowerFrontLeg
- removed joint Torso_BackLeg
- removed joint Torso_FrontLeg
- added joint B1_LB1: type revolute, parent B1, child LB1, origin xyz=0 -1 0 rpy=0 0 0, axis 1 0 0, limit lower=-3.14159 upper=3.14159 effort=0.0 velocity=0.0
- added joint F1_LF1: type revolute, parent F1, child LF1, origin xyz=0 1 0 rpy=0 0 0, axis 1 0 0, limit lower=-3.14159 upper=3.14159 effort=0.0 velocity=0.0
- added joint Torso_B1: type revolute, parent Torso, child B1, origin xyz=0 -0.5 1 rpy=0 0 0, axis 1 0 0, limit lower=-3.14159 upper=3.14159 effort=0.0 velocity=0.0
- added joint Torso_F1: type revolute, parent Torso, child F1, origin xyz=0 0.5 1 rpy=0 0 0, axis 1 0 0, limit lower=-3.14159 upper=3.14159 effort=0.0 velocity=0.0

Commit message: done for L number of leg pairs

File: body.urdf (robot description, URDF)
Before this commit: robot robot, 5 links, 4 joints
Links:
- added link B2, mass 1; collision box size=0.2 1 0.2; visual box size=0.2 1 0.2
- added link B3, mass 1; collision box size=0.2 1 0.2; visual box size=0.2 1 0.2
- added link B4, mass 1; collision box size=0.2 1 0.2; visual box size=0.2 1 0.2
- added link B5, mass 1; collision box size=0.2 1 0.2; visual box size=0.2 1 0.2
- added link F2, mass 1; collision box size=0.2 1 0.2; visual box size=0.2 1 0.2
- added link F3, mass 1; collision box size=0.2 1 0.2; visual box size=0.2 1 0.2
- added link F4, mass 1; collision box size=0.2 1 0.2; visual box size=0.2 1 0.2
- added link F5, mass 1; collision box size=0.2 1 0.2; visual box size=0.2 1 0.2
- added link LB2, mass 1; collision box size=0.2 0.2 1; visual box size=0.2 0.2 1
- added link LB3, mass 1; collision box size=0.2 0.2 1; visual box size=0.2 0.2 1
- added link LB4, mass 1; collision box size=0.2 0.2 1; visual box size=0.2 0.2 1
- added link LB5, mass 1; collision box size=0.2 0.2 1; visual box size=0.2 0.2 1
- added link LF2, mass 1; collision box size=0.2 0.2 1; visual box size=0.2 0.2 1
- added link LF3, mass 1; collision box size=0.2 0.2 1; visual box size=0.2 0.2 1
- added link LF4, mass 1; collision box size=0.2 0.2 1; visual box size=0.2 0.2 1
- added link LF5, mass 1; collision box size=0.2 0.2 1; visual box size=0.2 0.2 1
Joints:
- added joint B2_LB2: type revolute, parent B2, child LB2, origin xyz=0 -1 0 rpy=0 0 0, axis 1 0 0, limit lower=-3.14159 upper=3.14159 effort=0.0 velocity=0.0
- added joint B3_LB3: type revolute, parent B3, child LB3, origin xyz=0 -1 0 rpy=0 0 0, axis 1 0 0, limit lower=-3.14159 upper=3.14159 effort=0.0 velocity=0.0
- added joint B4_LB4: type revolute, parent B4, child LB4, origin xyz=0 -1 0 rpy=0 0 0, axis 1 0 0, limit lower=-3.14159 upper=3.14159 effort=0.0 velocity=0.0
- added joint B5_LB5: type revolute, parent B5, child LB5, origin xyz=0 -1 0 rpy=0 0 0, axis 1 0 0, limit lower=-3.14159 upper=3.14159 effort=0.0 velocity=0.0
- added joint F2_LF2: type revolute, parent F2, child LF2, origin xyz=0 1 0 rpy=0 0 0, axis 1 0 0, limit lower=-3.14159 upper=3.14159 effort=0.0 velocity=0.0
- added joint F3_LF3: type revolute, parent F3, child LF3, origin xyz=0 1 0 rpy=0 0 0, axis 1 0 0, limit lower=-3.14159 upper=3.14159 effort=0.0 velocity=0.0
- added joint F4_LF4: type revolute, parent F4, child LF4, origin xyz=0 1 0 rpy=0 0 0, axis 1 0 0, limit lower=-3.14159 upper=3.14159 effort=0.0 velocity=0.0
- added joint F5_LF5: type revolute, parent F5, child LF5, origin xyz=0 1 0 rpy=0 0 0, axis 1 0 0, limit lower=-3.14159 upper=3.14159 effort=0.0 velocity=0.0
- added joint Torso_B2: type revolute, parent Torso, child B2, origin xyz=0 -0.5 1 rpy=0 0 0, axis 1 0 0, limit lower=-3.14159 upper=3.14159 effort=0.0 velocity=0.0
- added joint Torso_B3: type revolute, parent Torso, child B3, origin xyz=0 -0.5 1 rpy=0 0 0, axis 1 0 0, limit lower=-3.14159 upper=3.14159 effort=0.0 velocity=0.0
- added joint Torso_B4: type revolute, parent Torso, child B4, origin xyz=0 -0.5 1 rpy=0 0 0, axis 1 0 0, limit lower=-3.14159 upper=3.14159 effort=0.0 velocity=0.0
- added joint Torso_B5: type revolute, parent Torso, child B5, origin xyz=0 -0.5 1 rpy=0 0 0, axis 1 0 0, limit lower=-3.14159 upper=3.14159 effort=0.0 velocity=0.0
- added joint Torso_F2: type revolute, parent Torso, child F2, origin xyz=0 0.5 1 rpy=0 0 0, axis 1 0 0, limit lower=-3.14159 upper=3.14159 effort=0.0 velocity=0.0
- added joint Torso_F3: type revolute, parent Torso, child F3, origin xyz=0 0.5 1 rpy=0 0 0, axis 1 0 0, limit lower=-3.14159 upper=3.14159 effort=0.0 velocity=0.0
- added joint Torso_F4: type revolute, parent Torso, child F4, origin xyz=0 0.5 1 rpy=0 0 0, axis 1 0 0, limit lower=-3.14159 upper=3.14159 effort=0.0 velocity=0.0
- added joint Torso_F5: type revolute, parent Torso, child F5, origin xyz=0 0.5 1 rpy=0 0 0, axis 1 0 0, limit lower=-3.14159 upper=3.14159 effort=0.0 velocity=0.0

Commit message: jumper finished

File: body.urdf (robot description, URDF)
Before this commit: robot robot, 21 links, 20 joints
Links:
- added link B10, mass 1; collision box size=0.2 1 0.2; visual box size=0.2 1 0.2
- added link B6, mass 1; collision box size=0.2 1 0.2; visual box size=0.2 1 0.2
- added link B7, mass 1; collision box size=0.2 1 0.2; visual box size=0.2 1 0.2
- added link B8, mass 1; collision box size=0.2 1 0.2; visual box size=0.2 1 0.2
- added link B9, mass 1; collision box size=0.2 1 0.2; visual box size=0.2 1 0.2
- added link F10, mass 1; collision box size=0.2 1 0.2; visual box size=0.2 1 0.2
- added link F6, mass 1; collision box size=0.2 1 0.2; visual box size=0.2 1 0.2
- added link F7, mass 1; collision box size=0.2 1 0.2; visual box size=0.2 1 0.2
- added link F8, mass 1; collision box size=0.2 1 0.2; visual box size=0.2 1 0.2
- added link F9, mass 1; collision box size=0.2 1 0.2; visual box size=0.2 1 0.2
- added link LB10, mass 1; collision box size=0.2 0.2 1; visual box size=0.2 0.2 1
- added link LB6, mass 1; collision box size=0.2 0.2 1; visual box size=0.2 0.2 1
- added link LB7, mass 1; collision box size=0.2 0.2 1; visual box size=0.2 0.2 1
- added link LB8, mass 1; collision box size=0.2 0.2 1; visual box size=0.2 0.2 1
- added link LB9, mass 1; collision box size=0.2 0.2 1; visual box size=0.2 0.2 1
- added link LF10, mass 1; collision box size=0.2 0.2 1; visual box size=0.2 0.2 1
- added link LF6, mass 1; collision box size=0.2 0.2 1; visual box size=0.2 0.2 1
- added link LF7, mass 1; collision box size=0.2 0.2 1; visual box size=0.2 0.2 1
- added link LF8, mass 1; collision box size=0.2 0.2 1; visual box size=0.2 0.2 1
- added link LF9, mass 1; collision box size=0.2 0.2 1; visual box size=0.2 0.2 1
Joints:
- added joint B10_LB10: type revolute, parent B10, child LB10, origin xyz=0 -1 0 rpy=0 0 0, axis 1 0 0, limit lower=-3.14159 upper=3.14159 effort=0.0 velocity=0.0
- added joint B6_LB6: type revolute, parent B6, child LB6, origin xyz=0 -1 0 rpy=0 0 0, axis 1 0 0, limit lower=-3.14159 upper=3.14159 effort=0.0 velocity=0.0
- added joint B7_LB7: type revolute, parent B7, child LB7, origin xyz=0 -1 0 rpy=0 0 0, axis 1 0 0, limit lower=-3.14159 upper=3.14159 effort=0.0 velocity=0.0
- added joint B8_LB8: type revolute, parent B8, child LB8, origin xyz=0 -1 0 rpy=0 0 0, axis 1 0 0, limit lower=-3.14159 upper=3.14159 effort=0.0 velocity=0.0
- added joint B9_LB9: type revolute, parent B9, child LB9, origin xyz=0 -1 0 rpy=0 0 0, axis 1 0 0, limit lower=-3.14159 upper=3.14159 effort=0.0 velocity=0.0
- added joint F10_LF10: type revolute, parent F10, child LF10, origin xyz=0 1 0 rpy=0 0 0, axis 1 0 0, limit lower=-3.14159 upper=3.14159 effort=0.0 velocity=0.0
- added joint F6_LF6: type revolute, parent F6, child LF6, origin xyz=0 1 0 rpy=0 0 0, axis 1 0 0, limit lower=-3.14159 upper=3.14159 effort=0.0 velocity=0.0
- added joint F7_LF7: type revolute, parent F7, child LF7, origin xyz=0 1 0 rpy=0 0 0, axis 1 0 0, limit lower=-3.14159 upper=3.14159 effort=0.0 velocity=0.0
- added joint F8_LF8: type revolute, parent F8, child LF8, origin xyz=0 1 0 rpy=0 0 0, axis 1 0 0, limit lower=-3.14159 upper=3.14159 effort=0.0 velocity=0.0
- added joint F9_LF9: type revolute, parent F9, child LF9, origin xyz=0 1 0 rpy=0 0 0, axis 1 0 0, limit lower=-3.14159 upper=3.14159 effort=0.0 velocity=0.0
- added joint Torso_B10: type revolute, parent Torso, child B10, origin xyz=0 -0.5 1 rpy=0 0 0, axis 1 0 0, limit lower=-3.14159 upper=3.14159 effort=0.0 velocity=0.0
- added joint Torso_B6: type revolute, parent Torso, child B6, origin xyz=0 -0.5 1 rpy=0 0 0, axis 1 0 0, limit lower=-3.14159 upper=3.14159 effort=0.0 velocity=0.0
- added joint Torso_B7: type revolute, parent Torso, child B7, origin xyz=0 -0.5 1 rpy=0 0 0, axis 1 0 0, limit lower=-3.14159 upper=3.14159 effort=0.0 velocity=0.0
- added joint Torso_B8: type revolute, parent Torso, child B8, origin xyz=0 -0.5 1 rpy=0 0 0, axis 1 0 0, limit lower=-3.14159 upper=3.14159 effort=0.0 velocity=0.0
- added joint Torso_B9: type revolute, parent Torso, child B9, origin xyz=0 -0.5 1 rpy=0 0 0, axis 1 0 0, limit lower=-3.14159 upper=3.14159 effort=0.0 velocity=0.0
- added joint Torso_F10: type revolute, parent Torso, child F10, origin xyz=0 0.5 1 rpy=0 0 0, axis 1 0 0, limit lower=-3.14159 upper=3.14159 effort=0.0 velocity=0.0
- added joint Torso_F6: type revolute, parent Torso, child F6, origin xyz=0 0.5 1 rpy=0 0 0, axis 1 0 0, limit lower=-3.14159 upper=3.14159 effort=0.0 velocity=0.0
- added joint Torso_F7: type revolute, parent Torso, child F7, origin xyz=0 0.5 1 rpy=0 0 0, axis 1 0 0, limit lower=-3.14159 upper=3.14159 effort=0.0 velocity=0.0
- added joint Torso_F8: type revolute, parent Torso, child F8, origin xyz=0 0.5 1 rpy=0 0 0, axis 1 0 0, limit lower=-3.14159 upper=3.14159 effort=0.0 velocity=0.0
- added joint Torso_F9: type revolute, parent Torso, child F9, origin xyz=0 0.5 1 rpy=0 0 0, axis 1 0 0, limit lower=-3.14159 upper=3.14159 effort=0.0 velocity=0.0

Commit message: cleaned up

File: body.urdf (robot description, URDF)
Before this commit: robot robot, 41 links, 40 joints
Links:
- removed link B10
- removed link B2
- removed link B3
- removed link B4
- removed link B5
- removed link B6
- removed link B7
- removed link B8
- removed link B9
- removed link F10
- removed link F2
- removed link F3
- removed link F4
- removed link F5
- removed link F6
- removed link F7
- removed link F8
- removed link F9
- removed link LB10
- removed link LB2
- removed link LB3
- removed link LB4
- removed link LB5
- removed link LB6
- removed link LB7
- removed link LB8
- removed link LB9
- removed link LF10
- removed link LF2
- removed link LF3
- removed link LF4
- removed link LF5
- removed link LF6
- removed link LF7
- removed link LF8
- removed link LF9
Joints:
- removed joint B10_LB10
- removed joint B2_LB2
- removed joint B3_LB3
- removed joint B4_LB4
- removed joint B5_LB5
- removed joint B6_LB6
- removed joint B7_LB7
- removed joint B8_LB8
- removed joint B9_LB9
- removed joint F10_LF10
- removed joint F2_LF2
- removed joint F3_LF3
- removed joint F4_LF4
- removed joint F5_LF5
- removed joint F6_LF6
- removed joint F7_LF7
- removed joint F8_LF8
- removed joint F9_LF9
- removed joint Torso_B10
- removed joint Torso_B2
- removed joint Torso_B3
- removed joint Torso_B4
- removed joint Torso_B5
- removed joint Torso_B6
- removed joint Torso_B7
- removed joint Torso_B8
- removed joint Torso_B9
- removed joint Torso_F10
- removed joint Torso_F2
- removed joint Torso_F3
- removed joint Torso_F4
- removed joint Torso_F5
- removed joint Torso_F6
- removed joint Torso_F7
- removed joint Torso_F8
- removed joint Torso_F9

Commit message: show initial worst

File: body.urdf (robot description, URDF)
Before this commit: robot robot, 5 links, 4 joints
Links:
- added link B2, mass 1; collision box size=0.2 1 0.2; visual box size=0.2 1 0.2
- added link B3, mass 1; collision box size=0.2 1 0.2; visual box size=0.2 1 0.2
- added link F2, mass 1; collision box size=0.2 1 0.2; visual box size=0.2 1 0.2
- added link F3, mass 1; collision box size=0.2 1 0.2; visual box size=0.2 1 0.2
- added link LB2, mass 1; collision box size=0.2 0.2 1; visual box size=0.2 0.2 1
- added link LB3, mass 1; collision box size=0.2 0.2 1; visual box size=0.2 0.2 1
- added link LF2, mass 1; collision box size=0.2 0.2 1; visual box size=0.2 0.2 1
- added link LF3, mass 1; collision box size=0.2 0.2 1; visual box size=0.2 0.2 1
Joints:
- added joint B2_LB2: type revolute, parent B2, child LB2, origin xyz=0 -1 0 rpy=0 0 0, axis 1 0 0, limit lower=-3.14159 upper=3.14159 effort=0.0 velocity=0.0
- added joint B3_LB3: type revolute, parent B3, child LB3, origin xyz=0 -1 0 rpy=0 0 0, axis 1 0 0, limit lower=-3.14159 upper=3.14159 effort=0.0 velocity=0.0
- added joint F2_LF2: type revolute, parent F2, child LF2, origin xyz=0 1 0 rpy=0 0 0, axis 1 0 0, limit lower=-3.14159 upper=3.14159 effort=0.0 velocity=0.0
- added joint F3_LF3: type revolute, parent F3, child LF3, origin xyz=0 1 0 rpy=0 0 0, axis 1 0 0, limit lower=-3.14159 upper=3.14159 effort=0.0 velocity=0.0
- added joint Torso_B2: type revolute, parent Torso, child B2, origin xyz=0 -0.5 1 rpy=0 0 0, axis 1 0 0, limit lower=-3.14159 upper=3.14159 effort=0.0 velocity=0.0
- added joint Torso_B3: type revolute, parent Torso, child B3, origin xyz=0 -0.5 1 rpy=0 0 0, axis 1 0 0, limit lower=-3.14159 upper=3.14159 effort=0.0 velocity=0.0
- added joint Torso_F2: type revolute, parent Torso, child F2, origin xyz=0 0.5 1 rpy=0 0 0, axis 1 0 0, limit lower=-3.14159 upper=3.14159 effort=0.0 velocity=0.0
- added joint Torso_F3: type revolute, parent Torso, child F3, origin xyz=0 0.5 1 rpy=0 0 0, axis 1 0 0, limit lower=-3.14159 upper=3.14159 effort=0.0 velocity=0.0

Commit message: mirrored legs to jump straight up, success!

File: body.urdf (robot description, URDF)
Before this commit: robot robot, 13 links, 12 joints
Links:
- added link B4, mass 1; collision box size=0.2 1 0.2; visual box size=0.2 1 0.2
- added link F4, mass 1; collision box size=0.2 1 0.2; visual box size=0.2 1 0.2
- added link LB4, mass 1; collision box size=0.2 0.2 1; visual box size=0.2 0.2 1
- added link LF4, mass 1; collision box size=0.2 0.2 1; visual box size=0.2 0.2 1
Joints:
- added joint B4_LB4: type revolute, parent B4, child LB4, origin xyz=0 -1 0 rpy=0 0 0, axis 1 0 0, limit lower=-3.14159 upper=3.14159 effort=0.0 velocity=0.0
- added joint F4_LF4: type revolute, parent F4, child LF4, origin xyz=0 1 0 rpy=0 0 0, axis 1 0 0, limit lower=-3.14159 upper=3.14159 effort=0.0 velocity=0.0
- added joint Torso_B4: type revolute, parent Torso, child B4, origin xyz=0 -0.5 1 rpy=0 0 0, axis 1 0 0, limit lower=-3.14159 upper=3.14159 effort=0.0 velocity=0.0
- added joint Torso_F4: type revolute, parent Torso, child F4, origin xyz=0 0.5 1 rpy=0 0 0, axis 1 0 0, limit lower=-3.14159 upper=3.14159 effort=0.0 velocity=0.0

Commit message: adding new body

File: body.urdf (robot description, URDF)
Before this commit: robot robot, 17 links, 16 joints
Links:
- removed link B2
- removed link B3
- removed link B4
- removed link F2
- removed link F3
- removed link F4
- removed link LB2
- removed link LB3
- removed link LB4
- removed link LF2
- removed link LF3
- removed link LF4
Joints:
- removed joint B2_LB2
- removed joint B3_LB3
- removed joint B4_LB4
- removed joint F2_LF2
- removed joint F3_LF3
- removed joint F4_LF4
- removed joint Torso_B2
- removed joint Torso_B3
- removed joint Torso_B4
- removed joint Torso_F2
- removed joint Torso_F3
- removed joint Torso_F4

Commit message: trying to run one simulation with new body

File: body.urdf (robot description, URDF)
Before this commit: robot robot, 5 links, 4 joints
Links:
- removed link B1
- removed link F1
- removed link LB1
- removed link LF1
Joints:
- removed joint B1_LB1
- removed joint F1_LF1
- removed joint Torso_B1
- removed joint Torso_F1

Commit message: snake body take 1

File: body.urdf (robot description, URDF)
Before this commit: robot robot, 9 links, 8 joints
Links:
- removed link BackLeg
- removed link FrontLeg
- removed link LeftLeg
- removed link LowerBackLeg
- removed link LowerFrontLeg
- removed link LowerLeftLeg
- removed link LowerRightLeg
- removed link RightLeg
- added link BL, mass 1; collision box size=1.1347780757924513 2.915510280578407 2.3706562108400258; visual box size=1.1347780757924513 2.915510280578407 2.3706562108400258
- link Torso: geometry collision box size=1.4266648176813996 2.6712573604426346 1.5589290880259083; visual box size=1.4266648176813996 2.6712573604426346 1.5589290880259083
Joints:
- removed joint BackLeg_LowerBackLeg
- removed joint FrontLeg_LowerFrontLeg
- removed joint LeftLeg_LowerLeftLeg
- removed joint RightLeg_LowerRightLeg
- removed joint Torso_BackLeg
- removed joint Torso_FrontLeg
- removed joint Torso_LeftLeg
- removed joint Torso_RightLeg
- added joint Torso_BL: type revolute, parent Torso, child BL, origin xyz=0 -0.5 1 rpy=0 0 0, axis 1 0 0, limit lower=-3.14159 upper=3.14159 effort=0.0 velocity=0.0

Commit message: 2 links

File: body.urdf (robot description, URDF)
Before this commit: robot robot, 2 links, 1 joints
Links:
- link BL: geometry collision box size=1 1 1; visual box size=1 1 1
- link Torso: geometry collision box size=2 2 2; visual box size=2 2 2
Joints:
- joint Torso_BL: origin xyz=0 -0.5 1 rpy=0 0 0 -> xyz=0 -1 0.5 rpy=0 0 0
