Commit message: random snake, need to randomize sensors

File: body.urdf (robot description, URDF)
Before this commit: robot robot, 2 links, 1 joints
Links:
- removed link BL
- removed link Torso
- added link 0, mass 1; collision box size=0.4045461276764989 1.4702028461291254 2.11434647954037; visual box size=0.4045461276764989 1.4702028461291254 2.11434647954037
- added link 1, mass 1; collision box size=2.664516069160475 1.1615786091444775 0.9389619630376511; visual box size=2.664516069160475 1.1615786091444775 0.9389619630376511
- added link 2, mass 1; collision box size=0.742274948904252 1.656712305367173 2.821916883271811; visual box size=0.742274948904252 1.656712305367173 2.821916883271811
- added link 3, mass 1; collision box size=1.4603423083043192 0.8216547400717122 1.4846835729641148; visual box size=1.4603423083043192 0.8216547400717122 1.4846835729641148
Joints:
- removed joint Torso_BL
- added joint 0_1: type revolute, parent 0, child 1, origin xyz=0 0.7351014230645627 2 rpy=0 0 0, axis 1 0 0, limit lower=-3.14159 upper=3.14159 effort=0.0 velocity=0.0
- added joint 1_2: type revolute, parent 1, child 2, origin xyz=0 1.1615786091444775 0 rpy=0 0 0, axis 1 0 0, limit lower=-3.14159 upper=3.14159 effort=0.0 velocity=0.0
- added joint 2_3: type revolute, parent 2, child 3, origin xyz=0 1.656712305367173 0 rpy=0 0 0, axis 1 0 0, limit lower=-3.14159 upper=3.14159 effort=0.0 velocity=0.0

Commit message: random color added

File: body.urdf (robot description, URDF)
Before this commit: robot robot, 4 links, 3 joints
Links:
- added link 4, mass 1; collision box size=2.5980708320247605 2.48536018950432 1.963383553181663; visual box size=2.5980708320247605 2.48536018950432 1.963383553181663
- added link 5, mass 1; collision box size=0.586479292639547 1.4441568082260736 0.3812950848523972; visual box size=0.586479292639547 1.4441568082260736 0.3812950848523972
- added link 6, mass 1; collision box size=2.452149747751129 0.8344718586260704 1.0026192876565636; visual box size=2.452149747751129 0.8344718586260704 1.0026192876565636
- link 0: geometry collision box size=2.1139091179911347 1.2716543287178443 0.8837326226774833; visual box size=2.1139091179911347 1.2716543287178443 0.8837326226774833
- link 1: geometry collision box size=1.7876115962979409 1.0506107569408936 1.6505070093349512; visual box size=1.7876115962979409 1.0506107569408936 1.6505070093349512
- link 2: geometry collision box size=0.9643157154818152 2.3379647372341466 2.3655593243536113; visual box size=0.9643157154818152 2.3379647372341466 2.3655593243536113
- link 3: geometry collision box size=2.395654772631027 1.5262719369221336 1.8066600553247547; visual box size=2.395654772631027 1.5262719369221336 1.8066600553247547
Joints:
- added joint 3_4: type revolute, parent 3, child 4, origin xyz=0 1.5262719369221336 0 rpy=0 0 0, axis 1 0 0, limit lower=-3.14159 upper=3.14159 effort=0.0 velocity=0.0
- added joint 4_5: type revolute, parent 4, child 5, origin xyz=0 2.48536018950432 0 rpy=0 0 0, axis 1 0 0, limit lower=-3.14159 upper=3.14159 effort=0.0 velocity=0.0
- added joint 5_6: type revolute, parent 5, child 6, origin xyz=0 1.4441568082260736 0 rpy=0 0 0, axis 1 0 0, limit lower=-3.14159 upper=3.14159 effort=0.0 velocity=0.0
- joint 0_1: origin xyz=0 0.7351014230645627 2 rpy=0 0 0 -> xyz=0 0.6358271643589222 2 rpy=0 0 0
- joint 1_2: origin xyz=0 1.1615786091444775 0 rpy=0 0 0 -> xyz=0 1.0506107569408936 0 rpy=0 0 0
- joint 2_3: origin xyz=0 1.656712305367173 0 rpy=0 0 0 -> xyz=0 2.3379647372341466 0 rpy=0 0 0

Commit message: random number + random sensors w/colors

File: body.urdf (robot description, URDF)
Before this commit: robot robot, 7 links, 6 joints
Links:
- removed link 2
- removed link 3
- removed link 4
- removed link 5
- removed link 6
- link 0: geometry collision box size=1.1235128720303857 1.7645095830070907 1.6881069937055795; visual box size=1.1235128720303857 1.7645095830070907 1.6881069937055795
- link 1: geometry collision box size=1.0715725804607492 1.4054618687310994 0.7655418034006269; visual box size=1.0715725804607492 1.4054618687310994 0.7655418034006269
Joints:
- removed joint 1_2
- removed joint 2_3
- removed joint 3_4
- removed joint 4_5
- removed joint 5_6
- joint 0_1: origin xyz=0 0.6358271643589222 2 rpy=0 0 0 -> xyz=0 0.8822547915035454 2 rpy=0 0 0

Commit message: done

File: body.urdf (robot description, URDF)
Before this commit: robot robot, 2 links, 1 joints
Links:
- added link 2, mass 1; collision box size=0.8338266424517349 1.4061927235928018 0.7910420299212051; visual box size=0.8338266424517349 1.4061927235928018 0.7910420299212051
- added link 3, mass 1; collision box size=1.416809869989379 1.4692236159635634 0.7709068211305832; visual box size=1.416809869989379 1.4692236159635634 0.7709068211305832
- added link 4, mass 1; collision box size=1.1981550614555752 0.6649679968240356 0.5524653328113053; visual box size=1.1981550614555752 0.6649679968240356 0.5524653328113053
- added link 5, mass 1; collision box size=0.9094067288692207 1.7150650861272694 1.6021758232883354; visual box size=0.9094067288692207 1.7150650861272694 1.6021758232883354
- added link 6, mass 1; collision box size=0.24936633969385152 1.3187687701255342 0.7813089564464535; visual box size=0.24936633969385152 1.3187687701255342 0.7813089564464535
- link 0: geometry collision box size=0.4963584240226255 0.984838801524289 1.5810861441228554; visual box size=0.4963584240226255 0.984838801524289 1.5810861441228554
- link 1: geometry collision box size=1.400134500899229 0.41534329926752306 0.3501651177555247; visual box size=1.400134500899229 0.41534329926752306 0.3501651177555247
Joints:
- added joint 1_2: type revolute, parent 1, child 2, origin xyz=0 0.41534329926752306 0 rpy=0 0 0, axis 1 0 0, limit lower=-3.14159 upper=3.14159 effort=0.0 velocity=0.0
- added joint 2_3: type revolute, parent 2, child 3, origin xyz=0 1.4061927235928018 0 rpy=0 0 0, axis 1 0 0, limit lower=-3.14159 upper=3.14159 effort=0.0 velocity=0.0
- added joint 3_4: type revolute, parent 3, child 4, origin xyz=0 1.4692236159635634 0 rpy=0 0 0, axis 1 0 0, limit lower=-3.14159 upper=3.14159 effort=0.0 velocity=0.0
- added joint 4_5: type revolute, parent 4, child 5, origin xyz=0 0.6649679968240356 0 rpy=0 0 0, axis 1 0 0, limit lower=-3.14159 upper=3.14159 effort=0.0 velocity=0.0
- added joint 5_6: type revolute, parent 5, child 6, origin xyz=0 1.7150650861272694 0 rpy=0 0 0, axis 1 0 0, limit lower=-3.14159 upper=3.14159 effort=0.0 velocity=0.0
- joint 0_1: origin xyz=0 0.8822547915035454 2 rpy=0 0 0 -> xyz=0 0.4924194007621445 1 rpy=0 0 0

Commit message: edit readme

File: body.urdf (robot description, URDF)
Before this commit: robot robot, 7 links, 6 joints
Links:
- removed link 5
- removed link 6
- link 0: geometry collision box size=0.41566671422776413 0.5276315390731015 0.7361874735866498; visual box size=0.41566671422776413 0.5276315390731015 0.7361874735866498
- link 1: geometry collision box size=0.7822570065624475 0.36128634423902195 1.6678430135035074; visual box size=0.7822570065624475 0.36128634423902195 1.6678430135035074
- link 2: geometry collision box size=0.7183627038668787 0.8939299502904736 1.258687664374084; visual box size=0.7183627038668787 0.8939299502904736 1.258687664374084
- link 3: geometry collision box size=1.631205117657767 0.9184429565221828 1.3069169074972853; visual box size=1.631205117657767 0.9184429565221828 1.3069169074972853
- link 4: geometry collision box size=1.9671993165968369 0.8496809687080704 0.7548705297378253; visual box size=1.9671993165968369 0.8496809687080704 0.7548705297378253
Joints:
- removed joint 4_5
- removed joint 5_6
- joint 0_1: origin xyz=0 0.4924194007621445 1 rpy=0 0 0 -> xyz=0 0.2638157695365507 1 rpy=0 0 0
- joint 1_2: origin xyz=0 0.41534329926752306 0 rpy=0 0 0 -> xyz=0 0.36128634423902195 0 rpy=0 0 0
- joint 2_3: origin xyz=0 1.4061927235928018 0 rpy=0 0 0 -> xyz=0 0.8939299502904736 0 rpy=0 0 0
- joint 3_4: origin xyz=0 1.4692236159635634 0 rpy=0 0 0 -> xyz=0 0.9184429565221828 0 rpy=0 0 0

Commit message: readme done

File: body.urdf (robot description, URDF)
Before this commit: robot robot, 5 links, 4 joints
Links:
- added link 5, mass 1; collision box size=1.1413375695869854 1.7224734819417657 1.0608727070324542; visual box size=1.1413375695869854 1.7224734819417657 1.0608727070324542
- added link 6, mass 1; collision box size=0.49124053588366534 1.7540786198239091 0.6138413301200274; visual box size=0.49124053588366534 1.7540786198239091 0.6138413301200274
- added link 7, mass 1; collision box size=1.7809065805898765 1.6744507352653308 1.0685007705254934; visual box size=1.7809065805898765 1.6744507352653308 1.0685007705254934
- added link 8, mass 1; collision box size=0.5260842816104785 0.4780831749128948 0.5709042519145177; visual box size=0.5260842816104785 0.4780831749128948 0.5709042519145177
- added link 9, mass 1; collision box size=1.1144712235672831 1.6883060507331644 0.5848833204097199; visual box size=1.1144712235672831 1.6883060507331644 0.5848833204097199
- link 0: geometry collision box size=0.43121540459998287 1.303720443511954 1.783074725718173; visual box size=0.43121540459998287 1.303720443511954 1.783074725718173
- link 1: geometry collision box size=0.2553192801223095 1.7539051757598534 1.210065899070172; visual box size=0.2553192801223095 1.7539051757598534 1.210065899070172
- link 2: geometry collision box size=0.29942820161614747 0.5263281800588808 0.3394193522707021; visual box size=0.29942820161614747 0.5263281800588808 0.3394193522707021
- link 3: geometry collision box size=0.730978617151794 0.913549522863216 0.8657315655329498; visual box size=0.730978617151794 0.913549522863216 0.8657315655329498
- link 4: geometry collision box size=1.440877203889347 0.9790596316521292 0.9950621374765609; visual box size=1.440877203889347 0.9790596316521292 0.9950621374765609
Joints:
- added joint 4_5: type revolute, parent 4, child 5, origin xyz=0 0.9790596316521292 0 rpy=0 0 0, axis 1 0 0, limit lower=-3.14159 upper=3.14159 effort=0.0 velocity=0.0
- added joint 5_6: type revolute, parent 5, child 6, origin xyz=0 1.7224734819417657 0 rpy=0 0 0, axis 1 0 0, limit lower=-3.14159 upper=3.14159 effort=0.0 velocity=0.0
- added joint 6_7: type revolute, parent 6, child 7, origin xyz=0 1.7540786198239091 0 rpy=0 0 0, axis 1 0 0, limit lower=-3.14159 upper=3.14159 effort=0.0 velocity=0.0
- added joint 7_8: type revolute, parent 7, child 8, origin xyz=0 1.6744507352653308 0 rpy=0 0 0, axis 1 0 0, limit lower=-3.14159 upper=3.14159 effort=0.0 velocity=0.0
- added joint 8_9: type revolute, parent 8, child 9, origin xyz=0 0.4780831749128948 0 rpy=0 0 0, axis 1 0 0, limit lower=-3.14159 upper=3.14159 effort=0.0 velocity=0.0
- joint 0_1: origin xyz=0 0.2638157695365507 1 rpy=0 0 0 -> xyz=0 0.651860221755977 1 rpy=0 0 0
- joint 1_2: origin xyz=0 0.36128634423902195 0 rpy=0 0 0 -> xyz=0 1.7539051757598534 0 rpy=0 0 0
- joint 2_3: origin xyz=0 0.8939299502904736 0 rpy=0 0 0 -> xyz=0 0.5263281800588808 0 rpy=0 0 0
- joint 3_4: origin xyz=0 0.9184429565221828 0 rpy=0 0 0 -> xyz=0 0.913549522863216 0 rpy=0 0 0

Commit message: first steps

File: body.urdf (robot description, URDF)
Before this commit: robot robot, 10 links, 9 joints
Links:
- removed link 2
- removed link 3
- removed link 4
- removed link 5
- removed link 6
- removed link 7
- removed link 8
- removed link 9
- link 0: geometry collision box size=1.811052737104687 0.9493833752200522 1.376093317632356; visual box size=1.811052737104687 0.9493833752200522 1.376093317632356
- link 1: geometry collision box size=1.4903822495513275 1.5778549907481751 1.552836050765438; visual box size=1.4903822495513275 1.5778549907481751 1.552836050765438
Joints:
- removed joint 1_2
- removed joint 2_3
- removed joint 3_4
- removed joint 4_5
- removed joint 5_6
- removed joint 6_7
- removed joint 7_8
- removed joint 8_9
- joint 0_1: origin xyz=0 0.651860221755977 1 rpy=0 0 0 -> xyz=0 0.4746916876100261 1 rpy=0 0 0

Commit message: adding multiple dimensions

File: body.urdf (robot description, URDF)
Before this commit: robot robot, 2 links, 1 joints
Links:
- added link 2, mass 1; collision box size=0.5287483097278922 1.7954616541182131 0.8749211086376494; visual box size=0.5287483097278922 1.7954616541182131 0.8749211086376494
- added link 3, mass 1; collision box size=1.828982700247914 1.2723612928784098 1.5629380458574897; visual box size=1.828982700247914 1.2723612928784098 1.5629380458574897
- added link 4, mass 1; collision box size=1.5177460547545631 1.2819411704023953 0.7108828636177786; visual box size=1.5177460547545631 1.2819411704023953 0.7108828636177786
- added link 5, mass 1; collision box size=0.5248870709996327 0.7009868391118987 1.9857926692007384; visual box size=0.5248870709996327 0.7009868391118987 1.9857926692007384
- link 0: geometry collision box size=0.821357529177938 0.627333337606889 1.097096795554876; visual box size=0.821357529177938 0.627333337606889 1.097096795554876
- link 1: geometry collision box size=1.366008166717816 1.0795660265145572 0.5541180417983304; visual box size=1.366008166717816 1.0795660265145572 0.5541180417983304
Joints:
- added joint 1_2: type revolute, parent 1, child 2, origin xyz=0 -1.0795660265145572 0 rpy=0 0 0, axis 1 0 0, limit lower=-3.14159 upper=3.14159 effort=0.0 velocity=0.0
- added joint 2_3: type revolute, parent 2, child 3, origin xyz=0 1.7954616541182131 0 rpy=0 0 0, axis 1 0 0, limit lower=-3.14159 upper=3.14159 effort=0.0 velocity=0.0
- added joint 3_4: type revolute, parent 3, child 4, origin xyz=-1.828982700247914 0 0 rpy=0 0 0, axis 1 0 0, limit lower=-3.14159 upper=3.14159 effort=0.0 velocity=0.0
- added joint 4_5: type revolute, parent 4, child 5, origin xyz=1.5177460547545631 0 0 rpy=0 0 0, axis 0 1 0, limit lower=-3.14159 upper=3.14159 effort=0.0 velocity=0.0
- joint 0_1: origin xyz=0 0.4746916876100261 1 rpy=0 0 0 -> xyz=0 0.3136666688034445 1 rpy=0 0 0

Commit message: changes

File: body.urdf (robot description, URDF)
Before this commit: robot robot, 6 links, 5 joints
Links:
- removed link 2
- removed link 3
- removed link 4
- removed link 5
- link 0: geometry collision box size=1 1 1; visual box size=1 1 1
- link 1: geometry collision box size=1 1 0.2; visual box size=1 1 0.2
Joints:
- removed joint 1_2
- removed joint 2_3
- removed joint 3_4
- removed joint 4_5
- joint 0_1: origin xyz=0 0.3136666688034445 1 rpy=0 0 0 -> xyz=0 0.5 0 rpy=0 0 0

Commit message: random choice of four directions

File: body.urdf (robot description, URDF)
Before this commit: robot robot, 2 links, 1 joints
Links:
- removed link 1
- added link 2, mass 1; collision box size=0.5 1 0.2; visual box size=0.5 1 0.2
Joints:
- removed joint 0_1
- added joint 0_2: type revolute, parent 0, child 2, origin xyz=-0.5 0 0.5 rpy=0 0 0, axis 1 1 0, limit lower=-3.14159 upper=3.14159 effort=0.0 velocity=0.0

Commit message: turtle looking thing

File: body.urdf (robot description, URDF)
Before this commit: robot robot, 2 links, 1 joints
Links:
- added link 1, mass 1; collision box size=0.5 1 0.2; visual box size=0.5 1 0.2
- added link 3, mass 1; collision box size=0.5 1 0.2; visual box size=0.5 1 0.2
- added link 4, mass 1; collision box size=0.5 1 0.2; visual box size=0.5 1 0.2
- link 0: geometry collision box size=2 1 0.5; visual box size=2 1 0.5
Joints:
- added joint 0_1: type revolute, parent 0, child 1, origin xyz=0.6666666666666666 0.5 0.25 rpy=0 0 0, axis 1 0 0, limit lower=-3.14159 upper=3.14159 effort=0.0 velocity=0.0
- added joint 0_3: type revolute, parent 0, child 3, origin xyz=-0.6666666666666666 -0.5 0.25 rpy=0 0 0, axis 1 0 0, limit lower=-3.14159 upper=3.14159 effort=0.0 velocity=0.0
- added joint 0_4: type revolute, parent 0, child 4, origin xyz=0.6666666666666666 -0.5 0.25 rpy=0 0 0, axis 1 0 0, limit lower=-3.14159 upper=3.14159 effort=0.0 velocity=0.0
- joint 0_2: axis 1 1 0 -> 1 0 0; origin xyz=-0.5 0 0.5 rpy=0 0 0 -> xyz=-0.6666666666666666 0.5 0.25 rpy=0 0 0

Commit message: frog

File: body.urdf (robot description, URDF)
Before this commit: robot robot, 5 links, 4 joints
Links:
- added link 11, mass 1; collision box size=0.9140226269504106 0.3604086055798218 0.2; visual box size=0.9140226269504106 0.3604086055798218 0.2
- added link 12, mass 1; collision box size=0.3539354774274408 0.33996765216175395 0.2; visual box size=0.3539354774274408 0.33996765216175395 0.2
- added link 13, mass 1; collision box size=0.6290032840483327 0.2802565460207325 0.2; visual box size=0.6290032840483327 0.2802565460207325 0.2
- added link 14, mass 1; collision box size=0.34213646916800955 0.39593118706885966 0.2; visual box size=0.34213646916800955 0.39593118706885966 0.2
- added link Head, mass 1; collision box size=0.5 0.5 0.5; visual box size=0.5 0.5 0.5
- link 0: geometry collision box size=1.6686860464787945 0.8210927181843265 0.42920778668377113; visual box size=1.6686860464787945 0.8210927181843265 0.42920778668377113
- link 1: geometry collision box size=0.1544180139353466 0.5949136461981945 0.09955146475771347; visual box size=0.1544180139353466 0.5949136461981945 0.09955146475771347
- link 2: geometry collision box size=0.36594601703753826 0.7361092702814549 0.16992401594049256; visual box size=0.36594601703753826 0.7361092702814549 0.16992401594049256
- link 3: geometry collision box size=0.3716448117658955 0.9345258470171619 0.06963637425655245; visual box size=0.3716448117658955 0.9345258470171619 0.06963637425655245
- link 4: geometry collision box size=0.3596440502291547 0.9856908161562861 0.06990749430674525; visual box size=0.3596440502291547 0.9856908161562861 0.06990749430674525
Joints:
- added joint 0_Head: type revolute, parent 0, child Head, origin xyz=-0.8343430232393972 0 0.21460389334188557 rpy=0 0 0, axis 0 1 0, limit lower=-3.14159 upper=3.14159 effort=0.0 velocity=0.0
- added joint 1_11: type revolute, parent 1, child 11, origin xyz=0.1544180139353466 0.5949136461981945 -0.049775732378856734 rpy=0 0 0, axis 0 1 0, limit lower=-3.14159 upper=3.14159 effort=0.0 velocity=0.0
- added joint 2_12: type revolute, parent 2, child 12, origin xyz=0 0.7361092702814549 -0.08496200797024628 rpy=0 0 0, axis 0 1 0, limit lower=-3.14159 upper=3.14159 effort=0.0 velocity=0.0
- added joint 3_13: type revolute, parent 3, child 13, origin xyz=0 -0.9345258470171619 -0.03481818712827622 rpy=0 0 0, axis 0 1 0, limit lower=-3.14159 upper=3.14159 effort=0.0 velocity=0.0
- added joint 4_14: type revolute, parent 4, child 14, origin xyz=0.3596440502291547 -0.9856908161562861 -0.03495374715337263 rpy=0 0 0, axis 0 1 0, limit lower=-3.14159 upper=3.14159 effort=0.0 velocity=0.0
- joint 0_1: origin xyz=0.6666666666666666 0.5 0.25 rpy=0 0 0 -> xyz=0.5562286821595982 0.41054635909216325 0.21460389334188557 rpy=0 0 0
- joint 0_2: origin xyz=-0.6666666666666666 0.5 0.25 rpy=0 0 0 -> xyz=-0.5562286821595982 0.41054635909216325 0.21460389334188557 rpy=0 0 0
- joint 0_3: origin xyz=-0.6666666666666666 -0.5 0.25 rpy=0 0 0 -> xyz=-0.5562286821595982 -0.41054635909216325 0.21460389334188557 rpy=0 0 0
- joint 0_4: origin xyz=0.6666666666666666 -0.5 0.25 rpy=0 0 0 -> xyz=0.5562286821595982 -0.41054635909216325 0.21460389334188557 rpy=0 0 0

Commit message: randomize
created a random choice to create a limb or not evaluated at each node

File: body.urdf (robot description, URDF)
Before this commit: robot robot, 10 links, 9 joints
Links:
- removed link 12
- removed link 14
- removed link 2
- link 0: geometry collision box size=1.6058574756338824 0.7109252497975546 0.344904265760399; visual box size=1.6058574756338824 0.7109252497975546 0.344904265760399
- link 1: geometry collision box size=0.48757783252261866 0.7597480266032486 0.15939332854443994; visual box size=0.48757783252261866 0.7597480266032486 0.15939332854443994
- link 11: geometry collision box size=0.5179730285880191 0.2456157668025786 0.2; visual box size=0.5179730285880191 0.2456157668025786 0.2
- link 13: geometry collision box size=0.5890670560005705 0.3922898323841182 0.2; visual box size=0.5890670560005705 0.3922898323841182 0.2
- link 3: geometry collision box size=0.13897416467289095 0.7757688007038513 0.05319588956239215; visual box size=0.13897416467289095 0.7757688007038513 0.05319588956239215
- link 4: geometry collision box size=0.38427163896162775 0.6741620703578325 0.09686614712268077; visual box size=0.38427163896162775 0.6741620703578325 0.09686614712268077
- link Head: geometry collision box size=0.4014643689084706 0.3554626248987773 0.25867819932029923; visual box size=0.4014643689084706 0.3554626248987773 0.25867819932029923
Joints:
- removed joint 0_2
- removed joint 2_12
- removed joint 4_14
- joint 0_1: origin xyz=0.5562286821595982 0.41054635909216325 0.21460389334188557 rpy=0 0 0 -> xyz=0.5352858252112941 0.3554626248987773 0.1724521328801995 rpy=0 0 0
- joint 0_3: origin xyz=-0.5562286821595982 -0.41054635909216325 0.21460389334188557 rpy=0 0 0 -> xyz=-0.5352858252112941 -0.3554626248987773 0.1724521328801995 rpy=0 0 0
- joint 0_4: origin xyz=0.5562286821595982 -0.41054635909216325 0.21460389334188557 rpy=0 0 0 -> xyz=0.5352858252112941 -0.3554626248987773 0.1724521328801995 rpy=0 0 0
- joint 0_Head: origin xyz=-0.8343430232393972 0 0.21460389334188557 rpy=0 0 0 -> xyz=-0.8029287378169412 0 0.1724521328801995 rpy=0 0 0
- joint 1_11: origin xyz=0.1544180139353466 0.5949136461981945 -0.049775732378856734 rpy=0 0 0 -> xyz=0.48757783252261866 0.7597480266032486 -0.07969666427221997 rpy=0 0 0
- joint 3_13: origin xyz=0 -0.9345258470171619 -0.03481818712827622 rpy=0 0 0 -> xyz=0 -0.7757688007038513 -0.026597944781196075 rpy=0 0 0
