Commit message: froggy

File: body.urdf (robot description, URDF)
Before this commit: robot robot, 7 links, 6 joints
Links:
- removed link 1
- removed link 11
- link 0: geometry collision box size=1.808077213006712 0.5508372319311375 0.23171970146262105; visual box size=1.808077213006712 0.5508372319311375 0.23171970146262105
- link 13: geometry collision box size=0.8094388939099528 0.18531171343174602 0.2; visual box size=0.8094388939099528 0.18531171343174602 0.2
- link 3: geometry collision box size=0.36469988647839835 0.6058724444532712 0.11628059880886528; visual box size=0.36469988647839835 0.6058724444532712 0.11628059880886528
- link 4: geometry collision box size=0.473464727351398 0.6253925906755732 0.12804781929346348; visual box size=0.473464727351398 0.6253925906755732 0.12804781929346348
- link Head: geometry collision box size=0.452019303251678 0.27541861596556877 0.17378977609696578; visual box size=0.452019303251678 0.27541861596556877 0.17378977609696578
Joints:
- removed joint 0_1
- removed joint 1_11
- joint 0_3: origin xyz=-0.5352858252112941 -0.3554626248987773 0.1724521328801995 rpy=0 0 0 -> xyz=-0.6026924043355707 -0.27541861596556877 0.11585985073131053 rpy=0 0 0
- joint 0_4: origin xyz=0.5352858252112941 -0.3554626248987773 0.1724521328801995 rpy=0 0 0 -> xyz=0.6026924043355707 -0.27541861596556877 0.11585985073131053 rpy=0 0 0
- joint 0_Head: origin xyz=-0.8029287378169412 0 0.1724521328801995 rpy=0 0 0 -> xyz=-0.904038606503356 0 0.11585985073131053 rpy=0 0 0
- joint 3_13: origin xyz=0 -0.7757688007038513 -0.026597944781196075 rpy=0 0 0 -> xyz=0 -0.6058724444532712 -0.05814029940443264 rpy=0 0 0

Commit message: frog/baby looking thing

File: body.urdf (robot description, URDF)
Before this commit: robot robot, 5 links, 4 joints
Links:
- added link 1, mass 1; collision box size=0.48598424256886796 0.40354823293515696 0.07554585138590511; visual box size=0.48598424256886796 0.40354823293515696 0.07554585138590511
- added link 11, mass 1; collision box size=0.35100195943542706 0.12890943664793014 0.10079675517589648; visual box size=0.35100195943542706 0.12890943664793014 0.10079675517589648
- added link 12, mass 1; collision box size=0.8002670406746908 0.20347564136647678 0.12023551787771582; visual box size=0.8002670406746908 0.20347564136647678 0.12023551787771582
- added link 14, mass 1; collision box size=0.5025363399759493 0.3799493863908271 0.196223640554595; visual box size=0.5025363399759493 0.3799493863908271 0.196223640554595
- added link 2, mass 1; collision box size=0.29360403639318666 0.6211438440207623 0.06558410229841254; visual box size=0.29360403639318666 0.6211438440207623 0.06558410229841254
- link 0: geometry collision box size=1.6779025369177505 1.4418202896009964 0.334041798704617; visual box size=1.6779025369177505 1.4418202896009964 0.334041798704617
- link 13: geometry collision box size=0.7813954800949665 0.36964873920413177 0.1453517639544379; visual box size=0.7813954800949665 0.36964873920413177 0.1453517639544379
- link 3: geometry collision box size=0.4303006459271702 0.4166806622779516 0.12249021800437744; visual box size=0.4303006459271702 0.4166806622779516 0.12249021800437744
- link 4: geometry collision box size=0.43259304334235915 0.6187796521464561 0.14939354792096216; visual box size=0.43259304334235915 0.6187796521464561 0.14939354792096216
- link Head: geometry collision box size=0.4194756342294376 0.7209101448004982 0.25053134902846275; visual box size=0.4194756342294376 0.7209101448004982 0.25053134902846275
Joints:
- added joint 0_1: type revolute, parent 0, child 1, origin xyz=0.5593008456392502 0.7209101448004982 0.1670208993523085 rpy=0 0 0, axis 1 0 0, limit lower=-3.14159 upper=3.14159 effort=0.0 velocity=0.0
- added joint 0_2: type revolute, parent 0, child 2, origin xyz=-0.5593008456392502 0.7209101448004982 0.1670208993523085 rpy=0 0 0, axis 1 0 0, limit lower=-3.14159 upper=3.14159 effort=0.0 velocity=0.0
- added joint 1_11: type revolute, parent 1, child 11, origin xyz=0.48598424256886796 0.40354823293515696 -0.037772925692952555 rpy=0 0 0, axis 0 1 0, limit lower=-3.14159 upper=3.14159 effort=0.0 velocity=0.0
- added joint 2_12: type revolute, parent 2, child 12, origin xyz=-0.29360403639318666 0.6211438440207623 -0.03279205114920627 rpy=0 0 0, axis 0 1 0, limit lower=-3.14159 upper=3.14159 effort=0.0 velocity=0.0
- added joint 4_14: type revolute, parent 4, child 14, origin xyz=0.43259304334235915 -0.6187796521464561 -0.07469677396048108 rpy=0 0 0, axis 0 1 0, limit lower=-3.14159 upper=3.14159 effort=0.0 velocity=0.0
- joint 0_3: origin xyz=-0.6026924043355707 -0.27541861596556877 0.11585985073131053 rpy=0 0 0 -> xyz=-0.5593008456392502 -0.7209101448004982 0.1670208993523085 rpy=0 0 0
- joint 0_4: origin xyz=0.6026924043355707 -0.27541861596556877 0.11585985073131053 rpy=0 0 0 -> xyz=0.5593008456392502 -0.7209101448004982 0.1670208993523085 rpy=0 0 0
- joint 0_Head: origin xyz=-0.904038606503356 0 0.11585985073131053 rpy=0 0 0 -> xyz=-0.8389512684588752 0 0.1670208993523085 rpy=0 0 0
- joint 3_13: origin xyz=0 -0.6058724444532712 -0.05814029940443264 rpy=0 0 0 -> xyz=-0.4303006459271702 -0.4166806622779516 -0.06124510900218872 rpy=0 0 0

Commit message: trying to add image to read me

File: body.urdf (robot description, URDF)
Before this commit: robot robot, 10 links, 9 joints
Links:
- link 0: geometry collision box size=1.5990969001439848 0.6947977524868147 0.47679136622384616; visual box size=1.5990969001439848 0.6947977524868147 0.47679136622384616
- link 1: geometry collision box size=0.16178359200199474 0.6254926826989647 0.05759044419181706; visual box size=0.16178359200199474 0.6254926826989647 0.05759044419181706
- link 11: geometry collision box size=0.3265935800447417 0.14738416879971275 0.11812524655330114; visual box size=0.3265935800447417 0.14738416879971275 0.11812524655330114
- link 12: geometry collision box size=0.3960714617241067 0.26197978576723535 0.07176767662410956; visual box size=0.3960714617241067 0.26197978576723535 0.07176767662410956
- link 13: geometry collision box size=0.8063127597601818 0.2967398252143598 0.056683607177486495; visual box size=0.8063127597601818 0.2967398252143598 0.056683607177486495
- link 14: geometry collision box size=0.6321262653322826 0.17280580121235922 0.055192298051390414; visual box size=0.6321262653322826 0.17280580121235922 0.055192298051390414
- link 2: geometry collision box size=0.10111570794985872 0.7496430712451854 0.13392528772596976; visual box size=0.10111570794985872 0.7496430712451854 0.13392528772596976
- link 3: geometry collision box size=0.32013710692504316 0.6504236790607496 0.129567216097683; visual box size=0.32013710692504316 0.6504236790607496 0.129567216097683
- link 4: geometry collision box size=0.23415035938281403 0.47640644324432896 0.156050472102652; visual box size=0.23415035938281403 0.47640644324432896 0.156050472102652
- link Head: geometry collision box size=0.3997742250359962 0.3473988762434074 0.35759352466788463; visual box size=0.3997742250359962 0.3473988762434074 0.35759352466788463
Joints:
- joint 0_1: origin xyz=0.5593008456392502 0.7209101448004982 0.1670208993523085 rpy=0 0 0 -> xyz=0.533032300047995 0.3473988762434074 0.23839568311192308 rpy=0 0 0
- joint 0_2: origin xyz=-0.5593008456392502 0.7209101448004982 0.1670208993523085 rpy=0 0 0 -> xyz=-0.533032300047995 0.3473988762434074 0.23839568311192308 rpy=0 0 0
- joint 0_3: origin xyz=-0.5593008456392502 -0.7209101448004982 0.1670208993523085 rpy=0 0 0 -> xyz=-0.533032300047995 -0.3473988762434074 0.23839568311192308 rpy=0 0 0
- joint 0_4: origin xyz=0.5593008456392502 -0.7209101448004982 0.1670208993523085 rpy=0 0 0 -> xyz=0.533032300047995 -0.3473988762434074 0.23839568311192308 rpy=0 0 0
- joint 0_Head: origin xyz=-0.8389512684588752 0 0.1670208993523085 rpy=0 0 0 -> xyz=-0.7995484500719924 0 0.23839568311192308 rpy=0 0 0
- joint 1_11: origin xyz=0.48598424256886796 0.40354823293515696 -0.037772925692952555 rpy=0 0 0 -> xyz=0.16178359200199474 0.6254926826989647 -0.02879522209590853 rpy=0 0 0
- joint 2_12: origin xyz=-0.29360403639318666 0.6211438440207623 -0.03279205114920627 rpy=0 0 0 -> xyz=-0.10111570794985872 0.7496430712451854 -0.06696264386298488 rpy=0 0 0
- joint 3_13: origin xyz=-0.4303006459271702 -0.4166806622779516 -0.06124510900218872 rpy=0 0 0 -> xyz=-0.32013710692504316 -0.6504236790607496 -0.0647836080488415 rpy=0 0 0
- joint 4_14: origin xyz=0.43259304334235915 -0.6187796521464561 -0.07469677396048108 rpy=0 0 0 -> xyz=0.23415035938281403 -0.47640644324432896 -0.078025236051326 rpy=0 0 0

Commit message: read me done, image worked

File: body.urdf (robot description, URDF)
Before this commit: robot robot, 10 links, 9 joints
Links:
- link 0: geometry collision box size=1.7653326837309282 0.9330913087447423 0.34469482709857957; visual box size=1.7653326837309282 0.9330913087447423 0.34469482709857957
- link 1: geometry collision box size=0.39225136093839674 0.7300352243475439 0.19156916721727657; visual box size=0.39225136093839674 0.7300352243475439 0.19156916721727657
- link 11: geometry collision box size=0.9731565850043471 0.21778330043574953 0.09663950428531355; visual box size=0.9731565850043471 0.21778330043574953 0.09663950428531355
- link 12: geometry collision box size=0.756656786596327 0.27205069903129775 0.10358955464026805; visual box size=0.756656786596327 0.27205069903129775 0.10358955464026805
- link 13: geometry collision box size=0.7666052811520203 0.26899193985731185 0.05963095569540902; visual box size=0.7666052811520203 0.26899193985731185 0.05963095569540902
- link 14: geometry collision box size=0.850865587369261 0.39859301576104633 0.16622574815110508; visual box size=0.850865587369261 0.39859301576104633 0.16622574815110508
- link 2: geometry collision box size=0.2882266256124013 0.7112056147620456 0.1602099911802476; visual box size=0.2882266256124013 0.7112056147620456 0.1602099911802476
- link 3: geometry collision box size=0.19317040053967696 0.7082237785411607 0.12009870312586189; visual box size=0.19317040053967696 0.7082237785411607 0.12009870312586189
- link 4: geometry collision box size=0.24478235897192846 0.7915420175783585 0.17058932772682456; visual box size=0.24478235897192846 0.7915420175783585 0.17058932772682456
- link Head: geometry collision box size=0.44133317093273206 0.46654565437237117 0.2585211203239347; visual box size=0.44133317093273206 0.46654565437237117 0.2585211203239347
Joints:
- joint 0_1: origin xyz=0.533032300047995 0.3473988762434074 0.23839568311192308 rpy=0 0 0 -> xyz=0.5884442279103094 0.46654565437237117 0.17234741354928979 rpy=0 0 0
- joint 0_2: origin xyz=-0.533032300047995 0.3473988762434074 0.23839568311192308 rpy=0 0 0 -> xyz=-0.5884442279103094 0.46654565437237117 0.17234741354928979 rpy=0 0 0
- joint 0_3: origin xyz=-0.533032300047995 -0.3473988762434074 0.23839568311192308 rpy=0 0 0 -> xyz=-0.5884442279103094 -0.46654565437237117 0.17234741354928979 rpy=0 0 0
- joint 0_4: origin xyz=0.533032300047995 -0.3473988762434074 0.23839568311192308 rpy=0 0 0 -> xyz=0.5884442279103094 -0.46654565437237117 0.17234741354928979 rpy=0 0 0
- joint 0_Head: origin xyz=-0.7995484500719924 0 0.23839568311192308 rpy=0 0 0 -> xyz=-0.8826663418654641 0 0.17234741354928979 rpy=0 0 0
- joint 1_11: origin xyz=0.16178359200199474 0.6254926826989647 -0.02879522209590853 rpy=0 0 0 -> xyz=0.39225136093839674 0.7300352243475439 -0.09578458360863829 rpy=0 0 0
- joint 2_12: origin xyz=-0.10111570794985872 0.7496430712451854 -0.06696264386298488 rpy=0 0 0 -> xyz=-0.2882266256124013 0.7112056147620456 -0.0801049955901238 rpy=0 0 0
- joint 3_13: origin xyz=-0.32013710692504316 -0.6504236790607496 -0.0647836080488415 rpy=0 0 0 -> xyz=-0.19317040053967696 -0.7082237785411607 -0.060049351562930946 rpy=0 0 0
- joint 4_14: origin xyz=0.23415035938281403 -0.47640644324432896 -0.078025236051326 rpy=0 0 0 -> xyz=0.24478235897192846 -0.7915420175783585 -0.08529466386341228 rpy=0 0 0

Commit message: done

File: body.urdf (robot description, URDF)
Before this commit: robot robot, 10 links, 9 joints
Links:
- link 0: geometry collision box size=1.5035625031299265 0.6417115535185957 0.30276268728831546; visual box size=1.5035625031299265 0.6417115535185957 0.30276268728831546
- link 1: geometry collision box size=0.3153206031535501 0.7888352690089179 0.07215272797711049; visual box size=0.3153206031535501 0.7888352690089179 0.07215272797711049
- link 11: geometry collision box size=0.3104607516885188 0.19924092292841364 0.12331063356672127; visual box size=0.3104607516885188 0.19924092292841364 0.12331063356672127
- link 12: geometry collision box size=0.33945558396809283 0.36224981283653535 0.06813715126272525; visual box size=0.33945558396809283 0.36224981283653535 0.06813715126272525
- link 13: geometry collision box size=0.7818168418160603 0.39533426216339007 0.06312003955505827; visual box size=0.7818168418160603 0.39533426216339007 0.06312003955505827
- link 14: geometry collision box size=0.4186924448564465 0.2823510869031574 0.1900046939984829; visual box size=0.4186924448564465 0.2823510869031574 0.1900046939984829
- link 2: geometry collision box size=0.31614989468268784 0.7332676991553537 0.10737531656413551; visual box size=0.31614989468268784 0.7332676991553537 0.10737531656413551
- link 3: geometry collision box size=0.418724347077316 0.7145614482302087 0.17745282481236718; visual box size=0.418724347077316 0.7145614482302087 0.17745282481236718
- link 4: geometry collision box size=0.47217358443714663 0.4068099326311807 0.16157688794225622; visual box size=0.47217358443714663 0.4068099326311807 0.16157688794225622
- link Head: geometry collision box size=0.3758906257824816 0.32085577675929783 0.2270720154662366; visual box size=0.3758906257824816 0.32085577675929783 0.2270720154662366
Joints:
- joint 0_1: origin xyz=0.5884442279103094 0.46654565437237117 0.17234741354928979 rpy=0 0 0 -> xyz=0.5011875010433088 0.32085577675929783 0.15138134364415773 rpy=0 0 0
- joint 0_2: origin xyz=-0.5884442279103094 0.46654565437237117 0.17234741354928979 rpy=0 0 0 -> xyz=-0.5011875010433088 0.32085577675929783 0.15138134364415773 rpy=0 0 0
- joint 0_3: origin xyz=-0.5884442279103094 -0.46654565437237117 0.17234741354928979 rpy=0 0 0 -> xyz=-0.5011875010433088 -0.32085577675929783 0.15138134364415773 rpy=0 0 0
- joint 0_4: origin xyz=0.5884442279103094 -0.46654565437237117 0.17234741354928979 rpy=0 0 0 -> xyz=0.5011875010433088 -0.32085577675929783 0.15138134364415773 rpy=0 0 0
- joint 0_Head: origin xyz=-0.8826663418654641 0 0.17234741354928979 rpy=0 0 0 -> xyz=-0.7517812515649632 0 0.15138134364415773 rpy=0 0 0
- joint 1_11: origin xyz=0.39225136093839674 0.7300352243475439 -0.09578458360863829 rpy=0 0 0 -> xyz=0.3153206031535501 0.7888352690089179 -0.036076363988555245 rpy=0 0 0
- joint 2_12: origin xyz=-0.2882266256124013 0.7112056147620456 -0.0801049955901238 rpy=0 0 0 -> xyz=-0.31614989468268784 0.7332676991553537 -0.05368765828206776 rpy=0 0 0
- joint 3_13: origin xyz=-0.19317040053967696 -0.7082237785411607 -0.060049351562930946 rpy=0 0 0 -> xyz=-0.418724347077316 -0.7145614482302087 -0.08872641240618359 rpy=0 0 0
- joint 4_14: origin xyz=0.24478235897192846 -0.7915420175783585 -0.08529466386341228 rpy=0 0 0 -> xyz=0.47217358443714663 -0.4068099326311807 -0.08078844397112811 rpy=0 0 0

Commit message: video taken

File: body.urdf (robot description, URDF)
Before this commit: robot robot, 10 links, 9 joints
Links:
- removed link 1
- removed link 11
- removed link 12
- removed link 13
- removed link 2
- removed link 3
- link 0: geometry collision box size=1.604453860444328 0.7299119179762191 0.4577791656402715; visual box size=1.604453860444328 0.7299119179762191 0.4577791656402715
- link 14: geometry collision box size=0.33141753552772374 0.37703994576566113 0.19622709524836046; visual box size=0.33141753552772374 0.37703994576566113 0.19622709524836046
- link 4: geometry collision box size=0.18349122336344106 0.7158120133266317 0.09001914789584986; visual box size=0.18349122336344106 0.7158120133266317 0.09001914789584986
- link Head: geometry collision box size=0.401113465111082 0.36495595898810956 0.34333437423020363; visual box size=0.401113465111082 0.36495595898810956 0.34333437423020363
Joints:
- removed joint 0_1
- removed joint 0_2
- removed joint 0_3
- removed joint 1_11
- removed joint 2_12
- removed joint 3_13
- joint 0_4: origin xyz=0.5011875010433088 -0.32085577675929783 0.15138134364415773 rpy=0 0 0 -> xyz=0.5348179534814427 -0.36495595898810956 0.22888958282013575 rpy=0 0 0
- joint 0_Head: origin xyz=-0.7517812515649632 0 0.15138134364415773 rpy=0 0 0 -> xyz=-0.802226930222164 0 0.22888958282013575 rpy=0 0 0
- joint 4_14: origin xyz=0.47217358443714663 -0.4068099326311807 -0.08078844397112811 rpy=0 0 0 -> xyz=0.18349122336344106 -0.7158120133266317 -0.04500957394792493 rpy=0 0 0

Commit message: makes legs 3d

File: body.urdf (robot description, URDF)
Before this commit: robot robot, 4 links, 3 joints
Links:
- removed link 14
- added link 13, mass 1; collision box size=0.4021020869870998 0.29716592797767766 0.06913411565152852; visual box size=0.4021020869870998 0.29716592797767766 0.06913411565152852
- added link 3, mass 1; collision box size=0.434709534856186 0.40019591507773355 0.992806749461099; visual box size=0.434709534856186 0.40019591507773355 0.992806749461099
- link 0: geometry collision box size=1.7368813887897647 0.9370360125644497 0.3418775712756221; visual box size=1.7368813887897647 0.9370360125644497 0.3418775712756221
- link 4: geometry collision box size=0.41500207587156845 0.43994698154081335 1.3800114322657437; visual box size=0.41500207587156845 0.43994698154081335 1.3800114322657437
- link Head: geometry collision box size=0.4342203471974412 0.46851800628222484 0.2564081784567166; visual box size=0.4342203471974412 0.46851800628222484 0.2564081784567166
Joints:
- removed joint 4_14
- added joint 0_3: type revolute, parent 0, child 3, origin xyz=-0.5789604629299215 -0.46851800628222484 0.17093878563781106 rpy=0 0 0, axis 0 1 0, limit lower=-3.14159 upper=3.14159 effort=0.0 velocity=0.0
- added joint 3_13: type revolute, parent 3, child 13, origin xyz=-0.434709534856186 -0.40019591507773355 -0.4964033747305495 rpy=0 0 0, axis 0 1 0, limit lower=-3.14159 upper=3.14159 effort=0.0 velocity=0.0
- joint 0_4: axis 1 0 0 -> 0 1 0; origin xyz=0.5348179534814427 -0.36495595898810956 0.22888958282013575 rpy=0 0 0 -> xyz=0.5789604629299215 -0.46851800628222484 0.17093878563781106 rpy=0 0 0
- joint 0_Head: origin xyz=-0.802226930222164 0 0.22888958282013575 rpy=0 0 0 -> xyz=-0.8684406943948824 0 0.17093878563781106 rpy=0 0 0

Commit message: fixed body, get off the floor

File: body.urdf (robot description, URDF)
Before this commit: robot robot, 5 links, 4 joints
Links:
- added link 1, mass 1; collision box size=0.3464544605358404 0.4685852543839522 0.7588028442504725; visual box size=0.3464544605358404 0.4685852543839522 0.7588028442504725
- added link 11, mass 1; collision box size=0.6218488918640307 0.3321474400320928 0.06631610955766386; visual box size=0.6218488918640307 0.3321474400320928 0.06631610955766386
- added link 12, mass 1; collision box size=0.751741061652093 0.3230317749264291 0.14670252013514634; visual box size=0.751741061652093 0.3230317749264291 0.14670252013514634
- added link 14, mass 1; collision box size=0.6072665567661321 0.20608779919415332 0.13098926316574325; visual box size=0.6072665567661321 0.20608779919415332 0.13098926316574325
- added link 2, mass 1; collision box size=0.49734865348493956 0.35426671749813465 1.2467548597939564; visual box size=0.49734865348493956 0.35426671749813465 1.2467548597939564
- link 0: geometry collision box size=1.5766223765158924 0.5348638523994884 0.3709218755914203; visual box size=1.5766223765158924 0.5348638523994884 0.3709218755914203
- link 13: geometry collision box size=0.5666272698398453 0.17210171573942312 0.1429857493518618; visual box size=0.5666272698398453 0.17210171573942312 0.1429857493518618
- link 3: geometry collision box size=0.20685966014342075 0.2709649582329222 0.6613907331801544; visual box size=0.20685966014342075 0.2709649582329222 0.6613907331801544
- link 4: geometry collision box size=0.26431242418413675 0.4639215446051211 1.3864147318596451; visual box size=0.26431242418413675 0.4639215446051211 1.3864147318596451
- link Head: geometry collision box size=0.3941555941289731 0.2674319261997442 0.3709218755914203; visual box size=0.3941555941289731 0.2674319261997442 0.3709218755914203
Joints:
- added joint 0_1: type revolute, parent 0, child 1, origin xyz=0.5255407921719641 0.2674319261997442 0.18546093779571016 rpy=0 0 0, axis 0 1 0, limit lower=-3.14159 upper=3.14159 effort=0.0 velocity=0.0
- added joint 0_2: type revolute, parent 0, child 2, origin xyz=-0.5255407921719641 0.2674319261997442 0.18546093779571016 rpy=0 0 0, axis 0 1 0, limit lower=-3.14159 upper=3.14159 effort=0.0 velocity=0.0
- added joint 1_11: type revolute, parent 1, child 11, origin xyz=0 0.4685852543839522 -0.7588028442504725 rpy=0 0 0, axis 0 1 0, limit lower=-3.14159 upper=3.14159 effort=0.0 velocity=0.0
- added joint 2_12: type revolute, parent 2, child 12, origin xyz=0 0.35426671749813465 -1.2467548597939564 rpy=0 0 0, axis 0 1 0, limit lower=-3.14159 upper=3.14159 effort=0.0 velocity=0.0
- added joint 4_14: type revolute, parent 4, child 14, origin xyz=0 -0.4639215446051211 -1.3864147318596451 rpy=0 0 0, axis 0 1 0, limit lower=-3.14159 upper=3.14159 effort=0.0 velocity=0.0
- joint 0_3: origin xyz=-0.5789604629299215 -0.46851800628222484 0.17093878563781106 rpy=0 0 0 -> xyz=-0.5255407921719641 -0.2674319261997442 0.18546093779571016 rpy=0 0 0
- joint 0_4: origin xyz=0.5789604629299215 -0.46851800628222484 0.17093878563781106 rpy=0 0 0 -> xyz=0.5255407921719641 -0.2674319261997442 0.18546093779571016 rpy=0 0 0
- joint 0_Head: origin xyz=-0.8684406943948824 0 0.17093878563781106 rpy=0 0 0 -> xyz=-0.7883111882579462 0 0.18546093779571016 rpy=0 0 0
- joint 3_13: origin xyz=-0.434709534856186 -0.40019591507773355 -0.4964033747305495 rpy=0 0 0 -> xyz=0 -0.2709649582329222 -0.6613907331801544 rpy=0 0 0
