Commit message: above floor now

File: body.urdf (robot description, URDF)
Before this commit: robot robot, 10 links, 9 joints
Links:
- link 0: geometry collision box size=1.5246597385110456 1.351286359156565 0.40174616503744076; visual box size=1.5246597385110456 1.351286359156565 0.40174616503744076
- link 1: geometry collision box size=0.2350064545446529 0.25674387279093247 1.1293252305467547; visual box size=0.2350064545446529 0.25674387279093247 1.1293252305467547
- link 11: geometry collision box size=0.5837383435954888 0.16503446137646938 0.11168922521813082; visual box size=0.5837383435954888 0.16503446137646938 0.11168922521813082
- link 12: geometry collision box size=0.5259585050819202 0.14393855113442916 0.11866439058115553; visual box size=0.5259585050819202 0.14393855113442916 0.11866439058115553
- link 13: geometry collision box size=0.7447405952097053 0.14193689995917824 0.1578280170288972; visual box size=0.7447405952097053 0.14193689995917824 0.1578280170288972
- link 14: geometry collision box size=0.3091946108597193 0.3501943815762293 0.15650593573691107; visual box size=0.3091946108597193 0.3501943815762293 0.15650593573691107
- link 2: geometry collision box size=0.4333375818502007 0.3202805198960813 1.3090500589977465; visual box size=0.4333375818502007 0.3202805198960813 1.3090500589977465
- link 3: geometry collision box size=0.2653660959567088 0.46367789534710735 0.6615538804414727; visual box size=0.2653660959567088 0.46367789534710735 0.6615538804414727
- link 4: geometry collision box size=0.25921244461593296 0.44767993737424994 1.3979669483906374; visual box size=0.25921244461593296 0.44767993737424994 1.3979669483906374
- link Head: geometry collision box size=0.3811649346277614 0.6756431795782825 0.40174616503744076; visual box size=0.3811649346277614 0.6756431795782825 0.40174616503744076
Joints:
- joint 0_1: origin xyz=0.5255407921719641 0.2674319261997442 0.18546093779571016 rpy=0 0 0 -> xyz=0.5082199128370152 0.6756431795782825 1.7008730825187204 rpy=0 0 0
- joint 0_2: origin xyz=-0.5255407921719641 0.2674319261997442 0.18546093779571016 rpy=0 0 0 -> xyz=-0.5082199128370152 0.6756431795782825 1.7008730825187204 rpy=0 0 0
- joint 0_3: origin xyz=-0.5255407921719641 -0.2674319261997442 0.18546093779571016 rpy=0 0 0 -> xyz=-0.5082199128370152 -0.6756431795782825 1.7008730825187204 rpy=0 0 0
- joint 0_4: origin xyz=0.5255407921719641 -0.2674319261997442 0.18546093779571016 rpy=0 0 0 -> xyz=0.5082199128370152 -0.6756431795782825 1.7008730825187204 rpy=0 0 0
- joint 0_Head: origin xyz=-0.7883111882579462 0 0.18546093779571016 rpy=0 0 0 -> xyz=-0.7623298692555228 0 1.7008730825187204 rpy=0 0 0
- joint 1_11: origin xyz=0 0.4685852543839522 -0.7588028442504725 rpy=0 0 0 -> xyz=0 0.25674387279093247 -1.1293252305467547 rpy=0 0 0
- joint 2_12: origin xyz=0 0.35426671749813465 -1.2467548597939564 rpy=0 0 0 -> xyz=0 0.3202805198960813 -1.3090500589977465 rpy=0 0 0
- joint 3_13: origin xyz=0 -0.2709649582329222 -0.6613907331801544 rpy=0 0 0 -> xyz=0 -0.46367789534710735 -0.6615538804414727 rpy=0 0 0
- joint 4_14: origin xyz=0 -0.4639215446051211 -1.3864147318596451 rpy=0 0 0 -> xyz=0 -0.44767993737424994 -1.3979669483906374 rpy=0 0 0

Commit message: fixed legs

File: body.urdf (robot description, URDF)
Before this commit: robot robot, 10 links, 9 joints
Links:
- link 0: geometry collision box size=1.5361753299712222 1.4089615043629968 0.37322162333270215; visual box size=1.5361753299712222 1.4089615043629968 0.37322162333270215
- link 1: geometry collision box size=0.15826807772089105 0.18406311793136015 1.3097833349009997; visual box size=0.15826807772089105 0.18406311793136015 1.3097833349009997
- link 11: geometry collision box size=0.545671483060189 0.18406311793136015 0.10363283717479756; visual box size=0.545671483060189 0.18406311793136015 0.10363283717479756
- link 12: geometry collision box size=0.6214003433296366 0.1309083078944703 0.12176704477004871; visual box size=0.6214003433296366 0.1309083078944703 0.12176704477004871
- link 13: geometry collision box size=0.6790302493296221 0.4198822456617073 0.13176310294773727; visual box size=0.6790302493296221 0.4198822456617073 0.13176310294773727
- link 14: geometry collision box size=0.5606211481764055 0.317136013781144 0.13033157447547855; visual box size=0.5606211481764055 0.317136013781144 0.13033157447547855
- link 2: geometry collision box size=0.48932039523535853 0.1309083078944703 1.2735516808570315; visual box size=0.48932039523535853 0.1309083078944703 1.2735516808570315
- link 3: geometry collision box size=0.42783446506809075 0.4198822456617073 1.0037599841577292; visual box size=0.42783446506809075 0.4198822456617073 1.0037599841577292
- link 4: geometry collision box size=0.30650295855446597 0.317136013781144 1.0270271253278875; visual box size=0.30650295855446597 0.317136013781144 1.0270271253278875
- link Head: geometry collision box size=0.38404383249280555 0.7044807521814984 0.37322162333270215; visual box size=0.38404383249280555 0.7044807521814984 0.37322162333270215
Joints:
- joint 0_1: origin xyz=0.5082199128370152 0.6756431795782825 1.7008730825187204 rpy=0 0 0 -> xyz=0.5120584433237407 0.7044807521814984 1.686610811666351 rpy=0 0 0
- joint 0_2: origin xyz=-0.5082199128370152 0.6756431795782825 1.7008730825187204 rpy=0 0 0 -> xyz=-0.5120584433237407 0.7044807521814984 1.686610811666351 rpy=0 0 0
- joint 0_3: origin xyz=-0.5082199128370152 -0.6756431795782825 1.7008730825187204 rpy=0 0 0 -> xyz=-0.5120584433237407 -0.7044807521814984 1.686610811666351 rpy=0 0 0
- joint 0_4: origin xyz=0.5082199128370152 -0.6756431795782825 1.7008730825187204 rpy=0 0 0 -> xyz=0.5120584433237407 -0.7044807521814984 1.686610811666351 rpy=0 0 0
- joint 0_Head: origin xyz=-0.7623298692555228 0 1.7008730825187204 rpy=0 0 0 -> xyz=-0.7680876649856111 0 1.686610811666351 rpy=0 0 0
- joint 1_11: origin xyz=0 0.25674387279093247 -1.1293252305467547 rpy=0 0 0 -> xyz=-0.07913403886044552 0.09203155896568008 -1.3097833349009997 rpy=0 0 0
- joint 2_12: origin xyz=0 0.3202805198960813 -1.3090500589977465 rpy=0 0 0 -> xyz=-0.24466019761767926 0.06545415394723515 -1.2735516808570315 rpy=0 0 0
- joint 3_13: origin xyz=0 -0.46367789534710735 -0.6615538804414727 rpy=0 0 0 -> xyz=-0.21391723253404538 -0.20994112283085364 -1.0037599841577292 rpy=0 0 0
- joint 4_14: origin xyz=0 -0.44767993737424994 -1.3979669483906374 rpy=0 0 0 -> xyz=-0.15325147927723298 -0.158568006890572 -1.0270271253278875 rpy=0 0 0

Commit message: legs same height now, too much variation

File: body.urdf (robot description, URDF)
Before this commit: robot robot, 10 links, 9 joints
Links:
- link 0: geometry collision box size=1.7088995036836667 0.7833207621128937 0.3648051419938493; visual box size=1.7088995036836667 0.7833207621128937 0.3648051419938493
- link 1: geometry collision box size=0.3298563603322683 0.4322179499041997 0.9; visual box size=0.3298563603322683 0.4322179499041997 0.9
- link 11: geometry collision box size=0.502968072399487 0.4322179499041997 0.1; visual box size=0.502968072399487 0.4322179499041997 0.1
- link 12: geometry collision box size=0.46206926829470607 0.19110113054786929 0.1; visual box size=0.46206926829470607 0.19110113054786929 0.1
- link 13: geometry collision box size=0.5497541712183874 0.45937059958135906 0.1; visual box size=0.5497541712183874 0.45937059958135906 0.1
- link 14: geometry collision box size=0.43695805414398414 0.307805109103266 0.1; visual box size=0.43695805414398414 0.307805109103266 0.1
- link 2: geometry collision box size=0.2539947990064919 0.19110113054786929 0.9; visual box size=0.2539947990064919 0.19110113054786929 0.9
- link 3: geometry collision box size=0.2752201789652581 0.45937059958135906 0.9; visual box size=0.2752201789652581 0.45937059958135906 0.9
- link 4: geometry collision box size=0.41327994140967095 0.307805109103266 0.9; visual box size=0.41327994140967095 0.307805109103266 0.9
- link Head: geometry collision box size=0.4272248759209167 0.39166038105644685 0.3648051419938493; visual box size=0.4272248759209167 0.39166038105644685 0.3648051419938493
Joints:
- joint 0_1: origin xyz=0.5120584433237407 0.7044807521814984 1.686610811666351 rpy=0 0 0 -> xyz=0.5696331678945555 0.39166038105644685 1.6824025709969246 rpy=0 0 0
- joint 0_2: origin xyz=-0.5120584433237407 0.7044807521814984 1.686610811666351 rpy=0 0 0 -> xyz=-0.5696331678945555 0.39166038105644685 1.6824025709969246 rpy=0 0 0
- joint 0_3: origin xyz=-0.5120584433237407 -0.7044807521814984 1.686610811666351 rpy=0 0 0 -> xyz=-0.5696331678945555 -0.39166038105644685 1.6824025709969246 rpy=0 0 0
- joint 0_4: origin xyz=0.5120584433237407 -0.7044807521814984 1.686610811666351 rpy=0 0 0 -> xyz=0.5696331678945555 -0.39166038105644685 1.6824025709969246 rpy=0 0 0
- joint 0_Head: origin xyz=-0.7680876649856111 0 1.686610811666351 rpy=0 0 0 -> xyz=-0.8544497518418334 0 1.6824025709969246 rpy=0 0 0
- joint 1_11: origin xyz=-0.07913403886044552 0.09203155896568008 -1.3097833349009997 rpy=0 0 0 -> xyz=-0.16492818016613414 0.21610897495209985 -0.9 rpy=0 0 0
- joint 2_12: origin xyz=-0.24466019761767926 0.06545415394723515 -1.2735516808570315 rpy=0 0 0 -> xyz=-0.12699739950324596 0.09555056527393464 -0.9 rpy=0 0 0
- joint 3_13: origin xyz=-0.21391723253404538 -0.20994112283085364 -1.0037599841577292 rpy=0 0 0 -> xyz=-0.13761008948262904 -0.22968529979067953 -0.9 rpy=0 0 0
- joint 4_14: origin xyz=-0.15325147927723298 -0.158568006890572 -1.0270271253278875 rpy=0 0 0 -> xyz=-0.20663997070483547 -0.153902554551633 -0.9 rpy=0 0 0

Commit message: mutate body each generation

File: body.urdf (robot description, URDF)
Before this commit: robot robot, 10 links, 9 joints
Links:
- removed link 1
- removed link 11
- removed link 13
- removed link 14
- removed link 3
- removed link 4
- link 0: geometry collision box size=1.6468356283999075 0.8987611450083047 0.3917720333837179; visual box size=1.6468356283999075 0.8987611450083047 0.3917720333837179
- link 12: geometry collision box size=0.521071994993083 0.21497906611173115 0.1; visual box size=0.521071994993083 0.21497906611173115 0.1
- link 2: geometry collision box size=0.2869048733881885 0.21497906611173115 0.9; visual box size=0.2869048733881885 0.21497906611173115 0.9
- link Head: geometry collision box size=0.4117089070999769 0.44938057250415236 0.3917720333837179; visual box size=0.4117089070999769 0.44938057250415236 0.3917720333837179
Joints:
- removed joint 0_1
- removed joint 0_3
- removed joint 0_4
- removed joint 1_11
- removed joint 3_13
- removed joint 4_14
- joint 0_2: origin xyz=-0.5696331678945555 0.39166038105644685 1.6824025709969246 rpy=0 0 0 -> xyz=-0.5489452094666358 0.44938057250415236 1.695886016691859 rpy=0 0 0
- joint 0_Head: origin xyz=-0.8544497518418334 0 1.6824025709969246 rpy=0 0 0 -> xyz=-0.8234178141999537 0 1.695886016691859 rpy=0 0 0
- joint 2_12: origin xyz=-0.12699739950324596 0.09555056527393464 -0.9 rpy=0 0 0 -> xyz=-0.14345243669409424 0.10748953305586557 -0.9 rpy=0 0 0

Commit message: generates new body each time

File: body.urdf (robot description, URDF)
Before this commit: robot robot, 4 links, 3 joints
Links:
- removed link 12
- removed link 2
- added link 1, mass 1; collision box size=0.3117724507662778 0.12848376140179602 0.9; visual box size=0.3117724507662778 0.12848376140179602 0.9
- added link 11, mass 1; collision box size=0.5263154412839164 0.12848376140179602 0.1; visual box size=0.5263154412839164 0.12848376140179602 0.1
- added link 13, mass 1; collision box size=0.580954908750341 0.3158873376844956 0.1; visual box size=0.580954908750341 0.3158873376844956 0.1
- added link 3, mass 1; collision box size=0.29482473845851576 0.3158873376844956 0.9; visual box size=0.29482473845851576 0.3158873376844956 0.9
- added link 4, mass 1; collision box size=0.3136321000469312 0.4041913562061551 0.9; visual box size=0.3136321000469312 0.4041913562061551 0.9
- link 0: geometry collision box size=1.6553195896802329 1.3041586720563596 0.27509877440870434; visual box size=1.6553195896802329 1.3041586720563596 0.27509877440870434
- link Head: geometry collision box size=0.4138298974200582 0.6520793360281798 0.27509877440870434; visual box size=0.4138298974200582 0.6520793360281798 0.27509877440870434
Joints:
- removed joint 0_2
- removed joint 2_12
- added joint 0_1: type revolute, parent 0, child 1, origin xyz=0.5517731965600776 0.6520793360281798 1.637549387204352 rpy=0 0 0, axis 0 1 0, limit lower=-3.14159 upper=3.14159 effort=0.0 velocity=0.0
- added joint 0_3: type revolute, parent 0, child 3, origin xyz=-0.5517731965600776 -0.6520793360281798 1.637549387204352 rpy=0 0 0, axis 0 1 0, limit lower=-3.14159 upper=3.14159 effort=0.0 velocity=0.0
- added joint 0_4: type revolute, parent 0, child 4, origin xyz=0.5517731965600776 -0.6520793360281798 1.637549387204352 rpy=0 0 0, axis 0 1 0, limit lower=-3.14159 upper=3.14159 effort=0.0 velocity=0.0
- added joint 1_11: type revolute, parent 1, child 11, origin xyz=-0.1558862253831389 0.06424188070089801 -0.9 rpy=0 0 0, axis 0 1 0, limit lower=-3.14159 upper=3.14159 effort=0.0 velocity=0.0
- added joint 3_13: type revolute, parent 3, child 13, origin xyz=-0.14741236922925788 -0.1579436688422478 -0.9 rpy=0 0 0, axis 0 1 0, limit lower=-3.14159 upper=3.14159 effort=0.0 velocity=0.0
- joint 0_Head: origin xyz=-0.8234178141999537 0 1.695886016691859 rpy=0 0 0 -> xyz=-0.8276597948401164 0 1.637549387204352 rpy=0 0 0

Commit message: parallel walker

File: body.urdf (robot description, URDF)
Before this commit: robot robot, 7 links, 6 joints
Links:
- removed link 1
- removed link 11
- removed link 13
- removed link 3
- removed link 4
- link 0: geometry collision box size=1.671956454300183 0.8462512511730396 0.45308817757347764; visual box size=1.671956454300183 0.8462512511730396 0.45308817757347764
- link Head: geometry collision box size=0.41798911357504576 0.4231256255865198 0.45308817757347764; visual box size=0.41798911357504576 0.4231256255865198 0.45308817757347764
Joints:
- removed joint 0_1
- removed joint 0_3
- removed joint 0_4
- removed joint 1_11
- removed joint 3_13
- joint 0_Head: origin xyz=-0.8276597948401164 0 1.637549387204352 rpy=0 0 0 -> xyz=-0.8359782271500915 0 1.726544088786739 rpy=0 0 0
