Commit message: no changes

File: body0.urdf (robot description, URDF)
Before this commit: robot robot, 6 links, 5 joints
Links:
- removed link 12
- removed link 13
- removed link 2
- removed link 3
- added link 1, mass 1; collision box size=0.16763633755718638 0.4309060041767099 0.9; visual box size=0.16763633755718638 0.4309060041767099 0.9
- added link 11, mass 1; collision box size=0.5380600077915983 0.4309060041767099 0.1; visual box size=0.5380600077915983 0.4309060041767099 0.1
- added link 14, mass 1; collision box size=0.590825717133105 0.3960079502296693 0.1; visual box size=0.590825717133105 0.3960079502296693 0.1
- added link 4, mass 1; collision box size=0.3953731802452449 0.3960079502296693 0.9; visual box size=0.3953731802452449 0.3960079502296693 0.9
- link 0: geometry collision box size=1.7678376970801635 0.9655239061429546 0.40933035209736807; visual box size=1.7678376970801635 0.9655239061429546 0.40933035209736807
- link Head: geometry collision box size=0.44195942427004087 0.4827619530714773 0.40933035209736807; visual box size=0.44195942427004087 0.4827619530714773 0.40933035209736807
Joints:
- removed joint 0_2
- removed joint 0_3
- removed joint 2_12
- removed joint 3_13
- added joint 0_1: type revolute, parent 0, child 1, origin xyz=0.5892792323600545 0.4827619530714773 1.004665176048684 rpy=0 0 0, axis 0 1 0, limit lower=-3.14159 upper=3.14159 effort=0.0 velocity=0.0
- added joint 0_4: type revolute, parent 0, child 4, origin xyz=0.5892792323600545 -0.4827619530714773 1.004665176048684 rpy=0 0 0, axis 0 1 0, limit lower=-3.14159 upper=3.14159 effort=0.0 velocity=0.0
- added joint 1_11: type revolute, parent 1, child 11, origin xyz=-0.08381816877859319 0.21545300208835494 -0.9 rpy=0 0 0, axis 0 1 0, limit lower=-3.14159 upper=3.14159 effort=0.0 velocity=0.0
- added joint 4_14: type revolute, parent 4, child 14, origin xyz=-0.19768659012262246 -0.19800397511483464 -0.9 rpy=0 0 0, axis 0 1 0, limit lower=-3.14159 upper=3.14159 effort=0.0 velocity=0.0
- joint 0_Head: origin xyz=-0.8729412663154796 0 1.0258888906243626 rpy=0 0 0 -> xyz=-0.8839188485400817 0 1.004665176048684 rpy=0 0 0
